Commit message: Tweak moments

File: bowl_6p25in_decomp/bowl_6p25in_decomp.urdf (robot description, URDF)
Before this commit: robot root, 12 links, 11 joints
Links:
- link link_bowl_6p25in_decomp_convex_piece_0: geometry collision mesh filename=bowl_6p25in_decomp_convex_piece_0.obj scale=1.0000E+00 1.0000E+00 1.0000E+00; visual mesh filename=bowl_6p25in_decomp_convex_piece_0.obj scale=1.0000E+00 1.0000E+00 1.0000E+00
- link link_bowl_6p25in_decomp_convex_piece_1: geometry collision mesh filename=bowl_6p25in_decomp_convex_piece_1.obj scale=1.0000E+00 1.0000E+00 1.0000E+00; visual mesh filename=bowl_6p25in_decomp_convex_piece_1.obj scale=1.0000E+00 1.0000E+00 1.0000E+00
- link link_bowl_6p25in_decomp_convex_piece_10: geometry collision mesh filename=bowl_6p25in_decomp_convex_piece_10.obj scale=1.0000E+00 1.0000E+00 1.0000E+00; visual mesh filename=bowl_6p25in_decomp_convex_piece_10.obj scale=1.0000E+00 1.0000E+00 1.0000E+00
- link link_bowl_6p25in_decomp_convex_piece_11: geometry collision mesh filename=bowl_6p25in_decomp_convex_piece_11.obj scale=1.0000E+00 1.0000E+00 1.0000E+00; visual mesh filename=bowl_6p25in_decomp_convex_piece_11.obj scale=1.0000E+00 1.0000E+00 1.0000E+00
- link link_bowl_6p25in_decomp_convex_piece_2: geometry collision mesh filename=bowl_6p25in_decomp_convex_piece_2.obj scale=1.0000E+00 1.0000E+00 1.0000E+00; visual mesh filename=bowl_6p25in_decomp_convex_piece_2.obj scale=1.0000E+00 1.0000E+00 1.0000E+00
- link link_bowl_6p25in_decomp_convex_piece_3: geometry collision mesh filename=bowl_6p25in_decomp_convex_piece_3.obj scale=1.0000E+00 1.0000E+00 1.0000E+00; visual mesh filename=bowl_6p25in_decomp_convex_piece_3.obj scale=1.0000E+00 1.0000E+00 1.0000E+00
- link link_bowl_6p25in_decomp_convex_piece_4: geometry collision mesh filename=bowl_6p25in_decomp_convex_piece_4.obj scale=1.0000E+00 1.0000E+00 1.0000E+00; visual mesh filename=bowl_6p25in_decomp_convex_piece_4.obj scale=1.0000E+00 1.0000E+00 1.0000E+00
- link link_bowl_6p25in_decomp_convex_piece_5: geometry collision mesh filename=bowl_6p25in_decomp_convex_piece_5.obj scale=1.0000E+00 1.0000E+00 1.0000E+00; visual mesh filename=bowl_6p25in_decomp_convex_piece_5.obj scale=1.0000E+00 1.0000E+00 1.0000E+00
- link link_bowl_6p25in_decomp_convex_piece_6: geometry collision mesh filename=bowl_6p25in_decomp_convex_piece_6.obj scale=1.0000E+00 1.0000E+00 1.0000E+00; visual mesh filename=bowl_6p25in_decomp_convex_piece_6.obj scale=1.0000E+00 1.0000E+00 1.0000E+00
- link link_bowl_6p25in_decomp_convex_piece_7: geometry collision mesh filename=bowl_6p25in_decomp_convex_piece_7.obj scale=1.0000E+00 1.0000E+00 1.0000E+00; visual mesh filename=bowl_6p25in_decomp_convex_piece_7.obj scale=1.0000E+00 1.0000E+00 1.0000E+00
- link link_bowl_6p25in_decomp_convex_piece_8: geometry collision mesh filename=bowl_6p25in_decomp_convex_piece_8.obj scale=1.0000E+00 1.0000E+00 1.0000E+00; visual mesh filename=bowl_6p25in_decomp_convex_piece_8.obj scale=1.0000E+00 1.0000E+00 1.0000E+00
- link link_bowl_6p25in_decomp_convex_piece_9: geometry collision mesh filename=bowl_6p25in_decomp_convex_piece_9.obj scale=1.0000E+00 1.0000E+00 1.0000E+00; visual mesh filename=bowl_6p25in_decomp_convex_piece_9.obj scale=1.0000E+00 1.0000E+00 1.0000E+00

File: plate_11in_decomp/plate_11in_decomp.urdf (robot description, URDF)
Before this commit: robot root, 8 links, 7 joints
Links:
- link link_plate_11in_decomp_convex_piece_0: geometry collision mesh filename=plate_11in_decomp_convex_piece_0.obj scale=1.0000E+00 1.0000E+00 1.0000E+00; visual mesh filename=plate_11in_decomp_convex_piece_0.obj scale=1.0000E+00 1.0000E+00 1.0000E+00
- link link_plate_11in_decomp_convex_piece_1: geometry collision mesh filename=plate_11in_decomp_convex_piece_1.obj scale=1.0000E+00 1.0000E+00 1.0000E+00; visual mesh filename=plate_11in_decomp_convex_piece_1.obj scale=1.0000E+00 1.0000E+00 1.0000E+00
- link link_plate_11in_decomp_convex_piece_2: geometry collision mesh filename=plate_11in_decomp_convex_piece_2.obj scale=1.0000E+00 1.0000E+00 1.0000E+00; visual mesh filename=plate_11in_decomp_convex_piece_2.obj scale=1.0000E+00 1.0000E+00 1.0000E+00
- link link_plate_11in_decomp_convex_piece_3: geometry collision mesh filename=plate_11in_decomp_convex_piece_3.obj scale=1.0000E+00 1.0000E+00 1.0000E+00; visual mesh filename=plate_11in_decomp_convex_piece_3.obj scale=1.0000E+00 1.0000E+00 1.0000E+00
- link link_plate_11in_decomp_convex_piece_4: geometry collision mesh filename=plate_11in_decomp_convex_piece_4.obj scale=1.0000E+00 1.0000E+00 1.0000E+00; visual mesh filename=plate_11in_decomp_convex_piece_4.obj scale=1.0000E+00 1.0000E+00 1.0000E+00
- link link_plate_11in_decomp_convex_piece_5: geometry collision mesh filename=plate_11in_decomp_convex_piece_5.obj scale=1.0000E+00 1.0000E+00 1.0000E+00; visual mesh filename=plate_11in_decomp_convex_piece_5.obj scale=1.0000E+00 1.0000E+00 1.0000E+00
- link link_plate_11in_decomp_convex_piece_6: geometry collision mesh filename=plate_11in_decomp_convex_piece_6.obj scale=1.0000E+00 1.0000E+00 1.0000E+00; visual mesh filename=plate_11in_decomp_convex_piece_6.obj scale=1.0000E+00 1.0000E+00 1.0000E+00
- link link_plate_11in_decomp_convex_piece_7: geometry collision mesh filename=plate_11in_decomp_convex_piece_7.obj scale=1.0000E+00 1.0000E+00 1.0000E+00; visual mesh filename=plate_11in_decomp_convex_piece_7.obj scale=1.0000E+00 1.0000E+00 1.0000E+00

File: plate_8p5in_decomp/plate_8p5in_decomp.urdf (robot description, URDF)
Before this commit: robot root, 8 links, 7 joints
Links:
- link link_plate_8p5in_decomp_convex_piece_0: geometry collision mesh filename=plate_8p5in_decomp_convex_piece_0.obj scale=1.0000E+00 1.0000E+00 1.0000E+00; visual mesh filename=plate_8p5in_decomp_convex_piece_0.obj scale=1.0000E+00 1.0000E+00 1.0000E+00
- link link_plate_8p5in_decomp_convex_piece_1: geometry collision mesh filename=plate_8p5in_decomp_convex_piece_1.obj scale=1.0000E+00 1.0000E+00 1.0000E+00; visual mesh filename=plate_8p5in_decomp_convex_piece_1.obj scale=1.0000E+00 1.0000E+00 1.0000E+00
- link link_plate_8p5in_decomp_convex_piece_2: geometry collision mesh filename=plate_8p5in_decomp_convex_piece_2.obj scale=1.0000E+00 1.0000E+00 1.0000E+00; visual mesh filename=plate_8p5in_decomp_convex_piece_2.obj scale=1.0000E+00 1.0000E+00 1.0000E+00
- link link_plate_8p5in_decomp_convex_piece_3: geometry collision mesh filename=plate_8p5in_decomp_convex_piece_3.obj scale=1.0000E+00 1.0000E+00 1.0000E+00; visual mesh filename=plate_8p5in_decomp_convex_piece_3.obj scale=1.0000E+00 1.0000E+00 1.0000E+00
- link link_plate_8p5in_decomp_convex_piece_4: geometry collision mesh filename=plate_8p5in_decomp_convex_piece_4.obj scale=1.0000E+00 1.0000E+00 1.0000E+00; visual mesh filename=plate_8p5in_decomp_convex_piece_4.obj scale=1.0000E+00 1.0000E+00 1.0000E+00
- link link_plate_8p5in_decomp_convex_piece_5: geometry collision mesh filename=plate_8p5in_decomp_convex_piece_5.obj scale=1.0000E+00 1.0000E+00 1.0000E+00; visual mesh filename=plate_8p5in_decomp_convex_piece_5.obj scale=1.0000E+00 1.0000E+00 1.0000E+00
- link link_plate_8p5in_decomp_convex_piece_6: geometry collision mesh filename=plate_8p5in_decomp_convex_piece_6.obj scale=1.0000E+00 1.0000E+00 1.0000E+00; visual mesh filename=plate_8p5in_decomp_convex_piece_6.obj scale=1.0000E+00 1.0000E+00 1.0000E+00
- link link_plate_8p5in_decomp_convex_piece_7: geometry collision mesh filename=plate_8p5in_decomp_convex_piece_7.obj scale=1.0000E+00 1.0000E+00 1.0000E+00; visual mesh filename=plate_8p5in_decomp_convex_piece_7.obj scale=1.0000E+00 1.0000E+00 1.0000E+00
